File: Single_transistor_AMP/Single_transistor_AMP.kicad_pcb (KiCad board)
At the start: 2 copper layers, 0 parts

Commit message: Majas darbs Nr.7
Parts:
- added C1: 1uF, Capacitor_THT:C_Rect_L4.0mm_W2.5mm_P2.50mm, F.Cu at (140.1, 108.3)
- added C2: 10uF, Capacitor_THT:C_Rect_L4.0mm_W2.5mm_P2.50mm, F.Cu at (140.1, 122.6)
- added C3: 1uF, Capacitor_THT:C_Rect_L4.0mm_W2.5mm_P2.50mm, F.Cu at (163.9, 113.0)
- added J1: Power_Supply, Connector_PinHeader_2.54mm:PinHeader_1x02_P2.54mm_Vertical, F.Cu at (137.6, 102.2)
- added J2: Uie, Connector_PinHeader_2.54mm:PinHeader_1x02_P2.54mm_Vertical, F.Cu at (140.1, 115.4)
- added J3: Uiz, Connector_PinHeader_2.54mm:PinHeader_1x02_P2.54mm_Vertical, F.Cu at (163.9, 120.0)
- added Q1: BC548, Package_TO_SOT_THT:TO-92_Inline, F.Cu at (162.2, 103.7)
- added R1: 33k, Resistor_THT:R_Axial_DIN0207_L6.3mm_D2.5mm_P10.16mm_Horizontal, F.Cu at (146.1, 107.5)
- added R2: 10k, Resistor_THT:R_Axial_DIN0207_L6.3mm_D2.5mm_P10.16mm_Horizontal, F.Cu at (156.2, 113.0)
- added R3: 3.3k, Resistor_THT:R_Axial_DIN0207_L6.3mm_D2.5mm_P10.16mm_Horizontal, F.Cu at (146.1, 102.2)
- added R4: 330, Resistor_THT:R_Axial_DIN0207_L6.3mm_D2.5mm_P10.16mm_Horizontal, F.Cu at (156.3, 117.9)
- added R5: 330, Resistor_THT:R_Axial_DIN0207_L6.3mm_D2.5mm_P10.16mm_Horizontal, F.Cu at (146.2, 122.6)
Other:
- board outline added: 37 x 29 mm

Commit message: Majas darbs Nr.8
Parts:
- moved R4 0.32 mm to (156.4, 118.2)
- moved R2 0.30 mm to (156.5, 112.9)
- moved R1 0.25 mm to (146.3, 107.5)
- moved R3 0.25 mm to (146.3, 102.2)
Routing:
- net Net-(C1-Pad1): track 0.00 -> 30.3 mm
- net Net-(C3-Pad2): track 0.00 -> 18.6 mm
- net Net-(Q1-Pad3): track 0.00 -> 15.6 mm
- net +10V: track 0.00 -> 11.2 mm
- net Net-(C2-Pad1): track 0.00 -> 10.5 mm
- net Net-(C1-Pad2): track 0.00 -> 7.05 mm
- net Net-(C3-Pad1): track 0.00 -> 7.00 mm
- added copper zone on B.Cu, net GND
- added copper zone on F.Cu, net GND
